File: schemat1/schemat.kicad_sch (KiCad schematic)
At the start: 10 parts, among them J2 Power Pins, Q5 NMOS

Commit message: zmiana footprinta tranzystora w układzie zabezpieczającym przed przeciwną polaryzacją
Parts:
- Q5: footprint Package_TO_SOT_THT:TO-92 -> Package_TO_SOT_THT:TO-220-3_Vertical
Changed lines of the file:
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@@
 			)
 		)
-		(property "Footprint" "Package_TO_SOT_THT:TO-92"
+		(property "Footprint" "Package_TO_SOT_THT:TO-220-3_Vertical"
 			(at 62.23 54.61 0)
 			(effects
