File: schemat1/game_logic.kicad_sch (KiCad schematic)
At the start: 4 parts, among them U4 4011, U8 74LS32

Commit message: poprawione schematy
Connections:
- net USER_1_VICTORY: now also U8.5; no longer U8.2
- net USER_2_VICTORY: now also U8.2; no longer U8.5
Changed lines of the file:
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@@
 	(paper "A4")
 	(junction
+		(at 184.15 62.23)
+		(diameter 0)
+		(color 0 0 0 0)
+	)
+	(junction
 		(at 210.82 104.14)
 		(diameter 0)
@@
 	)
 	(junction
-		(at 184.15 76.2)
-		(diameter 0)
-		(color 0 0 0 0)
-	)
-	(junction
 		(at 63.5 83.82)
 		(diameter 0)
@@
 	)
 	(junction
-		(at 184.15 127)
+		(at 184.15 113.03)
 		(diameter 0)
 		(color 0 0 0 0)
@@
 	(wire
 		(pts
-			(xy 184.15 127) (xy 127 127)
+			(xy 184.15 62.23) (xy 129.54 62.23)
 		)
 		(stroke
@@
 	(wire
 		(pts
-			(xy 127 53.34) (xy 137.16 53.34)
+			(xy 132.08 53.34) (xy 137.16 53.34)
 		)
 		(stroke
@@
 	(wire
 		(pts
-			(xy 127 76.2) (xy 127 53.34)
+			(xy 210.82 113.03) (xy 184.15 113.03)
+		)
+		(stroke
+			(width 0)
+			(type default)
+		)
+	)
+	(wire
+		(pts
+			(xy 129.54 62.23) (xy 129.54 104.14)
 		)
 		(stroke
@@
 	(wire
 		(pts
+			(xy 184.15 113.03) (xy 132.08 113.03)
+		)
+		(stroke
+			(width 0)
+			(type default)
+		)
+	)
+	(wire
+		(pts
 			(xy 63.5 25.4) (xy 63.5 43.18)
 		)
@@
 	(wire
 		(pts
+			(xy 132.08 53.34) (xy 132.08 113.03)
+		)
+		(stroke
+			(width 0)
+			(type default)
+		)
+	)
+	(wire
+		(pts
 			(xy 177.8 81.28) (xy 190.5 81.28)
 		)
@@
 	(wire
 		(pts
-			(xy 127 99.06) (xy 137.16 99.06)
+			(xy 121.92 99.06) (xy 137.16 99.06)
 		)
 		(stroke
@@
 	(wire
 		(pts
-			(xy 127 104.14) (xy 137.16 104.14)
-		)
-		(stroke
-			(width 0)
-			(type default)
-		)
-	)
-	(wire
-		(pts
-			(xy 210.82 104.14) (xy 210.82 113.03)
+			(xy 129.54 104.14) (xy 137.16 104.14)
 		)
 		(stroke
@@
 	(wire
 		(pts
-			(xy 127 48.26) (xy 137.16 48.26)
+			(xy 123.19 48.26) (xy 137.16 48.26)
 		)
 		(stroke
@@
 	(wire
 		(pts
-			(xy 184.15 76.2) (xy 127 76.2)
-		)
-		(stroke
-			(width 0)
-			(type default)
-		)
-	)
-	(wire
-		(pts
 			(xy 184.15 62.23) (xy 184.15 76.2)
 		)
@@
 	(wire
 		(pts
-			(xy 184.15 113.03) (xy 210.82 113.03)
+			(xy 210.82 62.23) (xy 184.15 62.23)
 		)
 		(stroke
@@
 	(wire
 		(pts
+			(xy 210.82 113.03) (xy 210.82 104.14)
+		)
+		(stroke
+			(width 0)
+			(type default)
+		)
+	)
+	(wire
+		(pts
 			(xy 181.61 64.77) (xy 181.61 55.88)
 		)
@@
 	(wire
 		(pts
-			(xy 127 127) (xy 127 104.14)
-		)
-		(stroke
-			(width 0)
-			(type default)
-		)
-	)
-	(wire
-		(pts
 			(xy 50.8 50.8) (xy 50.8 43.18)
-		)
-		(stroke
-			(width 0)
-			(type default)
-		)
-	)
-	(wire
-		(pts
-			(xy 184.15 62.23) (xy 210.82 62.23)
 		)
 		(stroke
@@
 	(hierarchical_label "~USER_1_SIGNAL"
 		(shape input)
-		(at 127 48.26 180)
+		(at 123.19 48.26 180)
 		(fields_autoplaced yes)
 		(effects
@@
 	(hierarchical_label "~USER_2_SIGNAL"
 		(shape input)
-		(at 127 99.06 180)
+		(at 121.92 99.06 180)
 		(fields_autoplaced yes)
 		(effects
