File: schemat1/led_lights.kicad_sch (KiCad schematic)
At the start: 6 parts

Commit message: poprawione schematy
Parts:
- R32, R33, R34: value 150R -> 100R
Changed lines of the file:
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@@
 			)
 		)
-		(property "Value" "150R"
+		(property "Value" "100R"
 			(at 90.17 97.79 90)
 			(effects
@@
 			)
 		)
-		(property "Value" "150R"
+		(property "Value" "100R"
 			(at 90.17 72.39 90)
 			(effects
@@
 			)
 		)
-		(property "Value" "150R"
+		(property "Value" "100R"
 			(at 90.17 46.99 90)
 			(effects
