File: schemat1/usr_interface.kicad_sch (KiCad schematic)
At the start: 9 parts, among them SW1 Player 1, SW2 Player 2, SW3 SW_Push

Commit message: poprawione schematy
Connections:
- no-connect marks 0 -> 1
Changed lines of the file:
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@@
 		(color 0 0 0 0)
+	)
+	(no_connect
+		(at 185.42 88.9)
 	)
 	(wire
