File: schemat1/schemat.kicad_pcb (KiCad board)
At the start: 2 copper layers, 100 x 100 mm, 91 parts, among them J1 Light Test Bridge, J2 Power Pins, Q1 BC547, Q2 BC547, Q3 BC547, Q4 BC547, Q5 NMOS, SW1 Player 1, SW2 Player 2, SW3 SW_Push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

Commit message: poprawione schematy
Parts:
- R32, R33, R34: value 150R -> 100R
Connections:
- U8 pad 2: /Licznik Czasu/USER_1_VICTORY -> /Licznik Czasu/USER_2_VICOTRY
- U8 pad 5: /Licznik Czasu/USER_2_VICOTRY -> /Licznik Czasu/USER_1_VICTORY
Routing:
- net /Licznik Czasu/USER_2_VICOTRY: track 83.7 -> 62.3 mm
- net /Licznik Czasu/USER_1_VICTORY: track 99.8 -> 88.6 mm
- net +5V: track 372.2 -> 373.8 mm
- net Net-(J2-Pin_2): track 6.62 -> 7.65 mm
Changed lines of the file:
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@@
 			)
 		)
-		(property "Value" "150R"
+		(property "Value" "100R"
 			(at 5.33 0 90)
 			(layer "F.SilkS")
@@
 			(layers "*.Cu" "*.Mask")
 			(remove_unused_layers no)
-			(net 60 "/Licznik Czasu/USER_1_VICTORY")
+			(net 61 "/Licznik Czasu/USER_2_VICOTRY")
 			(pintype "input")
 		)
@@
 			(layers "*.Cu" "*.Mask")
 			(remove_unused_layers no)
-			(net 61 "/Licznik Czasu/USER_2_VICOTRY")
+			(net 60 "/Licznik Czasu/USER_1_VICTORY")
 			(pintype "input")
 		)
@@
 			)
 		)
-		(property "Value" "150R"
+		(property "Value" "100R"
 			(at 5.08 0 90)
 			(layer "F.SilkS")
@@
 			)
 		)
-		(pad "1" thru_hole rect
-			(at 0 0 180)
-			(size 1.905 2)
+		(pad "1" thru_hole circle
+			(at 2.5 0 180)
+			(size 1.905 1.905)
 			(drill 1.1)
 			(layers "*.Cu" "*.Mask")
@@
 			(pintype "passive")
 		)
-		(pad "2" thru_hole oval
-			(at 2.54 0 180)
+		(pad "2" thru_hole rect
+			(at 0 0 180)
 			(size 1.905 2)
 			(drill 1.1)
@@
 			)
 		)
-		(property "Value" "150R"
+		(property "Value" "100R"
 			(at 5.08 0 90)
 			(layer "F.SilkS")
@@
 	)
 	(segment
+		(start 117.195 58.405)
+		(end 117.195 53.905)
+		(width 0.3)
+		(layer "F.Cu")
+		(net 2)
+	)
+	(segment
 		(start 112 53.57)
 		(end 114.64 53.57)
@@
 	)
 	(segment
-		(start 111 54.57)
-		(end 111 56)
-		(width 0.3)
-		(layer "F.Cu")
-		(net 2)
-	)
-	(segment
 		(start 74.68 71.56)
 		(end 79.38 76.26)
@@
 	)
 	(segment
-		(start 112 53.57)
-		(end 111 54.57)
-		(width 0.3)
-		(layer "F.Cu")
-		(net 2)
-	)
-	(segment
 		(start 104.75 50.195)
 		(end 101.375 53.57)
@@
 	)
 	(segment
-		(start 112.46 57.46)
-		(end 112.46 60.6)
-		(width 0.3)
-		(layer "F.Cu")
-		(net 2)
-	)
-	(segment
 		(start 33.34 102.8)
 		(end 33.34 98.4)
@@
 	)
 	(segment
+		(start 115 60.6)
+		(end 117.195 58.405)
+		(width 0.3)
+		(layer "F.Cu")
+		(net 2)
+	)
+	(segment
 		(start 104.75 33.33)
 		(end 95.83 33.33)
@@
 	)
 	(segment
+		(start 117.195 53.905)
+		(end 115.75 52.46)
+		(width 0.3)
+		(layer "F.Cu")
+		(net 2)
+	)
+	(segment
 		(start 33.42 82.95)
 		(end 33.42 87.8)
@@
 	)
 	(segment
-		(start 111 56)
-		(end 112.46 57.46)
-		(width 0.3)
-		(layer "F.Cu")
-		(net 2)
-	)
-	(segment
 		(start 33.32 103.2)
 		(end 33.32 102.82)
@@
 	)
 	(segment
-		(start 54.932448 38.14)
-		(end 56.372448 36.7)
-		(width 0.2)
-		(layer "B.Cu")
-		(net 60)
-	)
-	(segment
 		(start 50.94 39.85)
 		(end 49.84 38.75)
@@
 	)
 	(segment
-		(start 56.372448 29.04)
-		(end 56.372448 36.7)
-		(width 0.2)
-		(layer "B.Cu")
-		(net 60)
-	)
-	(segment
 		(start 108.25 50.99)
 		(end 101.54 57.7)
@@
 	)
 	(segment
-		(start 56.372448 29.04)
-		(end 57.472448 27.94)
-		(width 0.2)
-		(layer "B.Cu")
-		(net 60)
-	)
-	(segment
 		(start 50.94 45.27)
 		(end 53.82 45.27)
@@
 	)
 	(segment
-		(start 49.852448 27.94)
-		(end 46.2 31.592448)
-		(width 0.2)
-		(layer "F.Cu")
-		(net 61)
-	)
-	(segment
-		(start 46.2 31.592448)
-		(end 46.2 42.73)
-		(width 0.2)
-		(layer "F.Cu")
-		(net 61)
-	)
-	(segment
-		(start 46.2 42.73)
-		(end 49.84 46.37)
-		(width 0.2)
-		(layer "F.Cu")
-		(net 61)
-	)
-	(segment
 		(start 49.84 46.37)
 		(end 50.94 45.27)
@@
 	)
 	(segment
-		(start 116 55.5)
-		(end 115.5 55)
+		(start 112.5 60.6)
+		(end 112.5 58.25)
 		(width 0.3)
 		(layer "F.Cu")
@@
 	)
 	(segment
-		(start 115 60.6)
-		(end 115 55.75)
+		(start 116 55.5)
+		(end 115.5 55)
 		(width 0.3)
 		(layer "F.Cu")
@@
 	)
 	(segment
-		(start 115 55.75)
+		(start 112.5 58.25)
 		(end 115.75 55)
 		(width 0.3)
@@
 		(hatch edge 0.5)
 		(priority 2)
-		(connect_pads
+		(connect_pads yes
 			(clearance 0.5)
 		)

Commit message: gerbery
Parts:
- added G***: LOGO, LOGO, B.Cu at (60.8, 56.0)
- added G***: LOGO, LOGO, B.Cu at (89.8, 35.0)
- moved U14 0.12 mm to (116.8, 101.8)
Routing:
- net /Licznik Czasu/USER_2_VICOTRY: track 62.3 -> 81.8 mm
- net /Licznik Czasu/USER_1_VICTORY: track 88.6 -> 100.3 mm
- net Net-(U14-D): track 20.1 -> 20.8 mm
Other:
- board text added: "Grudzień 2024 Rewizja v1"
- board text added: "JLCJLCJLCJLC"
- board text added: "Może i wygląda jak *****, ale ważne, że działa."
